Commit message: Redone fanuc_moveit_config

File: fanuc_description/urdf/fanuc.urdf (robot description, URDF)
Before this commit: robot fanuc, 9 links, 8 joints
Links:
- removed link base
- added link world
- link base_link: mass None -> 0.1
Joints:
- removed joint base_link-base
- added joint base_link-world: type fixed, parent base_link, child world, origin xyz=0 0 0.450 rpy=0 0 0

Commit message: Some what working

File: fanuc_description/urdf/fanuc.urdf (robot description, URDF)
Before this commit: robot fanuc, 9 links, 8 joints
Links:
- added link base
Joints:
- removed joint base_link-world
- added joint base_link-base: type fixed, parent base_link, child base, origin xyz=0 0 0.450 rpy=0 0 0
- added joint world-base_link: type fixed, parent world, child base_link, origin xyz=0 0 0 rpy=0 0 0
